File: DCDC-Buck/COMPENSATOR.kicad_sch (KiCad schematic)
At the start: 0 parts

Commit message: Finishing SCH document.
Parts:
- added C3: 100nF, symbol Device:C
- added C4: 10nF, Capacitor_THT:C_Disc_D3.0mm_W2.0mm_P2.50mm, symbol Device:C
- added C5: 1nF, Capacitor_THT:C_Disc_D3.0mm_W2.0mm_P2.50mm, symbol Device:C
- added C6: 22nF, Capacitor_THT:C_Disc_D3.0mm_W2.0mm_P2.50mm, symbol Device:C
- added IC3: TL072, Package_DIP:DIP-8_W7.62mm_LongPads, symbol Amplifier_Operational:TL072
- added IC4: TL431ALP, Package_TO_SOT_THT:TO-92_Inline, symbol Reference_Voltage:TL431LP
- added LED1: L-317EGW, LED_THT:LED_D3.0mm, symbol Device:LED_Filled
- added R10: 220R, Resistor_THT:R_Axial_DIN0207_L6.3mm_D2.5mm_P7.62mm_Horizontal, symbol Device:R
- added R23: 100R, Resistor_THT:R_Axial_DIN0207_L6.3mm_D2.5mm_P7.62mm_Horizontal, symbol Device:R
- added R3, R4, R9: 10kR, Resistor_THT:R_Axial_DIN0207_L6.3mm_D2.5mm_P7.62mm_Horizontal, symbol Device:R
- added R5: 47R, Resistor_THT:R_Axial_DIN0207_L6.3mm_D2.5mm_P7.62mm_Horizontal, symbol Device:R
- added R6, R8: 3.9kR, Resistor_THT:R_Axial_DIN0207_L6.3mm_D2.5mm_P7.62mm_Horizontal, symbol Device:R
- added R7: 1kR, Resistor_THT:R_Axial_DIN0207_L6.3mm_D2.5mm_P7.62mm_Horizontal, symbol Device:R
Connections:
- net +15V: now also C3.1, IC3.8 (V+), R7.1, R8.2
- net +Vout: now also C4.1, R3.1
- net GND: now also C3.2, IC3.4 (V-), IC4.2 (A), R10.2, R4.2, R9.2
- net Verr: now also R23.1
- new net: C5.1, C6.1, IC3.7, R23.2
- new net: C5.2, IC3.6 (-), R3.2, R4.1, R5.2, R6.2
- new net: IC3.5 (+), IC4.1 (REF), IC4.3 (K), R7.2
- new net: C6.2, R6.1
- new net: IC3.3 (+), R8.1, R9.1
- new net: C4.2, R5.1
- new net: IC3.2 (-), LED1.1 (K), R10.1
- new net: IC3.1, LED1.2 (A)
Other:
- note added: "20mA"
- note added: "4.2V"
- title: (none) -> Compensator Type III

Commit message: Finishing PCB design with 2 layers.
Parts:
- removed R3: 10kR, Resistor_THT:R_Axial_DIN0207_L6.3mm_D2.5mm_P7.62mm_Horizontal, symbol Device:R
- added C16: 10uF, Capacitor_THT:C_Radial_D6.3mm_H11.0mm_P2.50mm, symbol Device:C_Polarized
- added RV1: 10kR, Potentiometer_THT:Potentiometer_Bourns_3296W_Vertical, symbol Device:R_Potentiometer_Trim
- C15: renamed from C3; footprint (none) -> Capacitor_THT:C_Disc_D3.0mm_W2.0mm_P2.50mm; Link https://www.multcomercial.com.br/capacitor-multicamada-100k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 -> https://www.multcomercial.com.br/capacitor-ceramico-disco-1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
- renumbered C5 to C12, C4 to C13, C6 to C14, IC3 to IC4, IC4 to IC5, R8 to R16, R6 to R17, R7 to R18, R9 to R19, R5 to R20, R23 to R21, R10 to R22, R4 to R23
Connections:
- net +15V: now also C16.1
- net +Vout: now also RV1.1, RV1.2
- net GND: now also C16.2
- net at C12.2, IC4.6 (-), R17.2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: now also RV1.3
- net Vref: now reaches IC4.5 (+), IC5.1 (REF), IC5.3 (K), R18.2
Other:
- moved on the sheet: C12, C13, C14, C15, IC4A, IC4B, IC4C, IC5, LED1, R16, R17, R18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
