File: DCDC-Buck/CONTROLLER.kicad_sch (KiCad schematic)
At the start: 0 parts

Commit message: Finishing SCH document.
Parts:
- added C7, C8: 100nF, symbol Device:C
- added IC5: TL074, Package_DIP:DIP-16_W7.62mm_LongPads, symbol Amplifier_Operational:TL074
- added R11, R12, R13, R14, R16, R17, R19, R20, R21: 10kR, Resistor_THT:R_Axial_DIN0207_L6.3mm_D2.5mm_P7.62mm_Horizontal, symbol Device:R
- added R15: 27kR, Resistor_THT:R_Axial_DIN0207_L6.3mm_D2.5mm_P7.62mm_Horizontal, symbol Device:R
- added R18: 2.2kR, Resistor_THT:R_Axial_DIN0207_L6.3mm_D2.5mm_P7.62mm_Horizontal, symbol Device:R
- added R22, R24: 100R, Resistor_THT:R_Axial_DIN0207_L6.3mm_D2.5mm_P7.62mm_Horizontal, symbol Device:R
Connections:
- net +15V: now also C8.1, IC5.11 (V-), R11.1, R16.1, R19.1
- net GND: now also C8.2, IC5.4 (V+), R12.2, R17.2, R20.2
- net Verr: now also IC5.12 (+)
- net Vpwm: now also R24.2
- new net: IC5.9 (-), R18.2, R21.1
- new net: IC5.8, R21.2, R22.1
- new net: IC5.3 (+), R13.1, R14.1
- new net: C7.2, IC5.7, R13.2, R18.1
- new net: IC5.5 (+), R16.2, R17.1
- new net: IC5.2 (-), R11.2, R12.1
- new net: IC5.10 (+), R19.2, R20.1
- new net: IC5.14, R24.1
- new net: IC5.1, R14.2, R15.1
- new net: C7.1, IC5.6 (-), R15.2
- new net Vtri: IC5.13 (-), R22.2

Commit message: Finishing PCB design with 2 layers.
Parts:
- added C11: 10uF, Capacitor_THT:C_Radial_D6.3mm_H11.0mm_P2.50mm, symbol Device:C_Polarized
- added C9: 100pF, Capacitor_THT:C_Disc_D3.0mm_W2.0mm_P2.50mm, symbol Device:C
- added unit 3 of IC3
- added unit 1 of IC3
- added unit 5 of IC3
- added unit 4 of IC3
- C10: renamed from C8; footprint (none) -> Capacitor_THT:C_Disc_D3.0mm_W2.0mm_P2.50mm; Link https://www.multcomercial.com.br/capacitor-multicamada-100k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 -> https://www.multcomercial.com.br/capacitor-ceramico-disco-1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
- C8: renamed from C7; value 100nF -> 390pF; footprint (none) -> Capacitor_THT:C_Disc_D3.0mm_W2.0mm_P2.50mm; Link https://www.multcomercial.com.br/capacitor-multicamada-100k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 -> https://www.multcomercial.com.br/capacitor-ceramico-disco-3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
- IC3: renamed from IC5; footprint Package_DIP:DIP-16_W7.62mm_LongPads -> Package_DIP:DIP-14_W7.62mm_LongPads
- R10: renamed from R24; value 100R -> 1kR
- renumbered R14 to R11, R17 to R12, R12 to R13, R13 to R14, R20 to R15, R21 to R3, R16 to R4, R11 to R5, R19 to R6, R15 to R7, R18 to R8, R22 to R9
Connections:
- net +15V: now also C11.1, IC3.11 (V-); no longer IC3.11 (V-)
- net GND: now also C11.2, C9.2, IC3.4 (V+); no longer IC3.4 (V+)
- net Verr: now also IC3.12 (+); no longer IC3.12 (+)
- net Vpwm: now also C9.1
- net Vtri: now also IC3.13 (-); no longer IC3.13 (-)
- net at R3.1, R8.2: now also IC3.9 (-); no longer IC3.9 (-)
- net at R3.2, R9.1: now also IC3.8; no longer IC3.8
- net at R11.1, R14.1: now also IC3.3 (+); no longer IC3.3 (+)
- net at R13.1, R5.2: now also IC3.2 (-); no longer IC3.2 (-)
- net at R15.1, R6.2: now also IC3.10 (+); no longer IC3.10 (+)
- net at R10.1: now also IC3.14; no longer IC3.14
- net at R11.2, R7.1: now also IC3.1; no longer IC3.1
Other:
- moved on the sheet: C10, C8, IC3B, R10, R11, R12, R13, R14, R15, R3, R4, R5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

Commit message: Fixing TL074 pinout issue, SCH revision is on date.
Connections:
- net +15V: now also IC3.4 (V+); no longer IC3.11 (V-)
- net GND: now also IC3.11 (V-); no longer IC3.4 (V+)
Changed lines of the file:
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@@
+	)
+	(symbol
+		(lib_id "Amplifier_Operational:TL074")
+		(at 100.33 133.35 0)
+		(mirror y)
+		(unit 5)
+		(body_style 1)
+		(exclude_from_sim no)
+		(in_bom yes)
+		(on_board yes)
+		(in_pos_files yes)
+		(dnp no)
+		(property "Reference" "IC3"
+			(at 96.266 132.588 0)
+			(show_name no)
+			(do_not_autoplace no)
+			(effects
+				(font
+					(size 1.27 1.27)
+				)
+				(justify right)
+			)
+		)
+		(property "Value" "TL074"
+			(at 96.266 134.62 0)
+			(show_name no)
+			(do_not_autoplace no)
+			(effects
+				(font
+					(size 1.27 1.27)
+				)
+				(justify right)
+			)
+		)
+		(property "Footprint" "Package_DIP:DIP-14_W7.62mm_LongPads"
+			(at 101.6 130.81 0)
+			(hide yes)
+			(show_name no)
+			(do_not_autoplace no)
+			(effects
+				(font
+					(size 1.27 1.27)
+				)
+			)
+		)
+		(property "Datasheet" "http://www.ti.com/lit/ds/symlink/tl071.pdf"
+			(at 99.06 128.27 0)
+			(hide yes)
+			(show_name no)
+			(do_not_autoplace no)
+			(effects
+				(font
+					(size 1.27 1.27)
+				)
+			)
+		)
+		(property "Description" "Quad Low-Noise JFET-Input Operational Amplifiers, DIP-14/SOIC-14"
+			(at 100.33 133.35 0)
+			(hide yes)
+			(show_name no)
+			(do_not_autoplace no)
+			(effects
+				(font
+					(size 1.27 1.27)
+				)
+			)
+		)
+		(pin "1"
+		)
+		(pin "2"
+		)
+		(pin "5"
+		)
+		(pin "7"
+		)
+		(pin "10"
+		)
+		(pin "6"
+		)
+		(pin "8"
+		)
+		(pin "13"
+		)
+		(pin "9"
+		)
+		(pin "14"
+		)
+		(pin "4"
+		)
+		(pin "3"
+		)
+		(pin "12"
+		)
+		(pin "11"
+		)
+		(instances
+			(project "DCDC-Buck"
+				(path "/959e3d1c-01d0-4c7d-bf19-165b598aa596/b4854b56-cd62-46e7-9f3e-c4c93ab06a71"
+					(reference "IC3")
+					(unit 5)
+				)
+			)
+		)
 	)
 	(symbol
@@
 				)
 			)
-		)
-	)
-	(symbol
-		(lib_id "Amplifier_Operational:TL074")
-		(at 105.41 133.35 0)
-		(mirror x)
-		(unit 5)
-		(body_style 1)
-		(exclude_from_sim no)
-		(in_bom yes)
-		(on_board yes)
-		(in_pos_files yes)
-		(dnp no)
-		(fields_autoplaced yes)
-		(property "Reference" "IC3"
-			(at 101.6 132.0799 0)
-			(show_name no)
-			(do_not_autoplace no)
-			(effects
-				(font
-					(size 1.27 1.27)
-				)
-				(justify right)
-			)
-		)
-		(property "Value" "TL074"
-			(at 101.6 134.6199 0)
-			(show_name no)
-			(do_not_autoplace no)
-			(effects
-				(font
-					(size 1.27 1.27)
-				)
-				(justify right)
-			)
-		)
-		(property "Footprint" "Package_DIP:DIP-14_W7.62mm_LongPads"
-			(at 104.14 135.89 0)
-			(hide yes)
-			(show_name no)
-			(do_not_autoplace no)
-			(effects
-				(font
-					(size 1.27 1.27)
-				)
-			)
-		)
-		(property "Datasheet" "http://www.ti.com/lit/ds/symlink/tl071.pdf"
-			(at 106.68 138.43 0)
-			(hide yes)
-			(show_name no)
-			(do_not_autoplace no)
-			(effects
-				(font
-					(size 1.27 1.27)
-				)
-			)
-		)
-		(property "Description" "Quad Low-Noise JFET-Input Operational Amplifiers, DIP-14/SOIC-14"
-			(at 105.41 133.35 0)
-			(hide yes)
-			(show_name no)
-			(do_not_autoplace no)
-			(effects
-				(font
-					(size 1.27 1.27)
-				)
-			)
-		)
-		(pin "1"
-		)
-		(pin "2"
-		)
-		(pin "5"
-		)
-		(pin "7"
-		)
-		(pin "10"
-		)
-		(pin "6"
-		)
-		(pin "8"
-		)
-		(pin "13"
-		)
-		(pin "9"
-		)
-		(pin "14"
-		)
-		(pin "4"
-		)
-		(pin "3"
-		)
-		(pin "12"
-		)
-		(pin "11"
-		)
-		(instances
-			(project "DCDC-Buck"
-				(path "/959e3d1c-01d0-4c7d-bf19-165b598aa596/b4854b56-cd62-46e7-9f3e-c4c93ab06a71"
-					(reference "IC3")
-					(unit 5)
-				)
-			)

Commit message: Editing some bug fixes in controller and plant.
Parts:
- C8: value 390pF -> 1nF
- R11: value 10kR -> 27kR
- R3: value 10kR -> 4.7kR
Changed lines of the file:
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@@
 			)
 		)
-		(property "Value" "10kR"
+		(property "Value" "4.7kR"
 			(at 173.736 82.5499 90)
 			(show_name no)
@@
 			)
 		)
-		(property "Value" "390pF"
+		(property "Value" "1nF"
 			(at 125.222 81.28 90)
 			(show_name no)
@@
 			)
 		)
-		(property "Value" "10kR"
+		(property "Value" "27kR"
 			(at 84.836 101.5999 90)
 			(show_name no)

Commit message: Validating and verifying bug fix in controller, ready for v1.0.1  release.
Parts:
- R3: value 4.7kR -> 10kR
- R8: value 2.2kR -> 10kR
Changed lines of the file:
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@@
 			)
 		)
-		(property "Value" "4.7kR"
+		(property "Value" "10kR"
 			(at 173.736 82.5499 90)
 			(show_name no)
@@
 			)
 		)
-		(property "Value" "2.2kR"
+		(property "Value" "10kR"
 			(at 158.242 83.058 90)
 			(show_name no)

Commit message: Changing 1nF capacitor and buck-plant inductor footprints. Ready to release v1.0.1 (bug-fixes).
Parts:
- C8: footprint Capacitor_THT:C_Disc_D3.0mm_W2.0mm_P2.50mm -> Capacitor_THT:C_Rect_L7.2mm_W3.5mm_P5.00mm_FKS2_FKP2_MKS2_MKP2
Changed lines of the file:
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@@
 			)
 		)
-		(property "Footprint" "Capacitor_THT:C_Disc_D3.0mm_W2.0mm_P2.50mm"
+		(property "Footprint" "Capacitor_THT:C_Rect_L7.2mm_W3.5mm_P5.00mm_FKS2_FKP2_MKS2_MKP2"
 			(at 133.35 76.5048 0)
 			(hide yes)
