File: DCDC-Buck/DCDC-Buck.kicad_pcb (KiCad board)
At the start: 2 copper layers, 94 x 70 mm, 61 parts, among them CN1 STLZ950GH, CN2 STLZ950GH, IC1 LM7815CT, IC2 IR2117, IC3 TL074, IC4 TL072, IC5 TL431ALP, Q1 IRF740

Commit message: FInishing BOM and PCB.
Parts:
- C1: footprint Capacitor_THT:C_Disc_D3.0mm_W2.0mm_P2.50mm -> Capacitor_THT:C_Rect_L10.0mm_W5.0mm_P5.00mm_P7.50mm
- R1: value 100 -> 100R
- moved C2 2.37 mm to (48.2, 58.0)
- moved C1 1.45 mm to (51.2, 73.2)
- moved D1 1.25 mm to (51.2, 68.6)
Routing:
- net +15V: track 235.4 -> 231.1 mm
- net GND: vias 65 -> 69

Commit message: Revision A is ok to build!
Connections:
- IC3 pad 11: +15V -> GND
- IC3 pad 4: GND -> +15V
Routing:
- net +15V: track 231.1 -> 231.7 mm
Changed lines of the file:
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@@
 		(grid_origin 36.75 105.5)
 		(pcbplotparams
-			(layerselection 0x00000000_00000000_55555555_5755f5ff)
+			(layerselection 0x00000000_00000000_55555555_57555555)
 			(plot_on_all_layers_selection 0x00000000_00000000_00000000_00000000)
 			(disableapertmacros no)
-			(usegerberextensions no)
+			(usegerberextensions yes)
 			(usegerberattributes yes)
-			(usegerberadvancedattributes yes)
-			(creategerberjobfile yes)
+			(usegerberadvancedattributes no)
+			(creategerberjobfile no)
 			(dashed_line_dash_ratio 12)
 			(dashed_line_gap_ratio 3)
@@
 			(plotframeref no)
 			(mode 1)
-			(useauxorigin no)
+			(useauxorigin yes)
 			(pdf_front_fp_property_popups yes)
 			(pdf_back_fp_property_popups yes)
@@
 			(plotpadnumbers no)
 			(hidednponfab no)
-			(sketchdnponfab yes)
-			(crossoutdnponfab yes)
+			(sketchdnponfab no)
+			(crossoutdnponfab no)
 			(subtractmaskfromsilk no)
 			(outputformat 1)
 			(mirror no)
-			(drillshape 1)
+			(drillshape 0)
 			(scaleselection 1)
 			(outputdirectory "")
@@
 		(tags "THT DIP DIL PDIP 2.54mm 7.62mm 300mil LongPads")
 		(property "Reference" "IC3"
-			(at 3.81 7.62 0)
+			(at 0.62 -2.71 0)
 			(layer "F.SilkS")
 			(effects
@@
 			(layers "*.Cu" "*.Mask")
 			(remove_unused_layers no)
-			(net "GND")
+			(net "+15V")
 			(pinfunction "V+_4")
 			(pintype "power_in")
@@
 			(layers "*.Cu" "*.Mask")
 			(remove_unused_layers no)
-			(net "+15V")
+			(net "GND")
 			(pinfunction "V-_11")
 			(pintype "power_in")
@@
 		(sheetname "/INPUT/")
 		(sheetfile "INPUT.kicad_sch")
+		(units
+			(unit
+				(name "A")
+				(pins "1" "2")
+			)
+		)
 		(attr through_hole)
 		(duplicate_pad_numbers_are_jumpers no)
@@
 		(sheetname "/INPUT/")
 		(sheetfile "INPUT.kicad_sch")
+		(units
+			(unit
+				(name "A")
+				(pins "1" "2")
+			)
+		)
 		(attr through_hole)
 		(duplicate_pad_numbers_are_jumpers no)
@@
 	)
 	(segment
-		(start 95.5 47)
-		(end 93.75 45.25)
+		(start 96.92 56.17)
+		(end 95.5 54.75)
 		(width 1)
 		(layer "B.Cu")
@@
 	)
 	(segment
-		(start 92 56.17)
-		(end 94.08 56.17)
+		(start 99.62 56.17)
+		(end 96.92 56.17)
 		(width 1)
 		(layer "B.Cu")
@@
 	)
 	(segment
-		(start 95.5 54.75)
-		(end 95.5 47)
-		(width 1)
-		(layer "B.Cu")
-		(net "+15V")
-	)
-	(segment
 		(start 87.5 43.5)
 		(end 89.25 45.25)
@@
 	)
 	(segment
-		(start 94.08 56.17)
-		(end 95.5 54.75)
-		(width 1)
-		(layer "B.Cu")
-		(net "+15V")
-	)
-	(segment
 		(start 83 67.67)
 		(end 93.59 67.67)
@@
 	)
 	(segment
+		(start 95.5 47)
+		(end 93.75 45.25)
+		(width 1)
+		(layer "B.Cu")
+		(net "+15V")
+	)
+	(segment
 		(start 69.42 64.08)
 		(end 71.5 62)
@@
 	)
 	(segment
+		(start 95.5 54.75)
+		(end 95.5 47)
+		(width 1)
+		(layer "B.Cu")
+		(net "+15V")
+	)
+	(segment
 		(start 69 46.25)
 		(end 77.25 46.25)
@@
 	)
 	(via
+		(at 90 56.25)
+		(size 0.8)
+		(drill 0.4)
+		(layers "F.Cu" "B.Cu")
+		(free yes)
+		(net "GND")
+	)
+	(via
 		(at 40.25 59.33)
 		(size 0.8)
@@
 	)
 	(via
-		(at 97.5 57.33)
-		(size 0.8)
-		(drill 0.4)
-		(layers "F.Cu" "B.Cu")
-		(free yes)
-		(net "GND")
-	)
-	(via
 		(at 45.5 56.08)
 		(size 0.8)
@@
 	)
 	(via
-		(at 81.25 65.83)
+		(at 94.005567 56.25)
 		(size 0.8)
 		(drill 0.4)
@@
 	)
 	(via
-		(at 72.25 74.83)
+		(at 81.25 65.83)
 		(size 0.8)
 		(drill 0.4)
@@
 	)
 	(via
-		(at 127 85.83)
+		(at 72.25 74.83)
 		(size 0.8)
 		(drill 0.4)
@@
 	)
 	(via
-		(at 97.5 55.08)
+		(at 127 85.83)
 		(size 0.8)
 		(drill 0.4)
@@
 	)
 	(zone
+		(net "+15V")
+		(layer "B.Cu")
+		(hatch none 0.1)
+		(priority 30025)
+		(attr
+			(teardrop
+				(type padvia)
+			)
+		)
+		(connect_pads yes
+			(clearance 0)
+		)
+		(min_thickness 0.0254)
+		(fill yes
+			(island_removal_mode 1)
+		)
+		(polygon
+			(pts
+				(xy 94.525094 46.7322) (xy 95.2322 46.025094) (xy 94.368408 44.742485) (xy 93.746569 45.246569)
+				(xy 93.242485 45.868408)
+			)
+		)
+	)
+	(zone
 		(net "Net-(IC4A--)")
 		(layer "B.Cu")
@@
 		(layer "B.Cu")
 		(hatch none 0.1)
-		(priority 30126)
+		(priority 30000)
 		(attr
 			(teardrop
@@
 		(polygon
 			(pts
-				(xy 51.53524 58.841867) (xy 50.828133 58.13476) (xy 51.888793 59.195421) (xy 50.47289 59.19711)
-				(xy 50.474581 57.781207)
+				(xy 49.41392 59.548973) (xy 50.121027 60.25608) (xy 51.636874 59.447339) (xy 51.253105 58.416895)
+				(xy 50.222659 58.033127)
 			)
 		)
@@
 		(layer "B.Cu")
 		(hatch none 0.1)
-		(priority 30000)
+		(priority 30126)
 		(attr
 			(teardrop
@@
 		(polygon
 			(pts
-				(xy 49.41392 59.548973) (xy 50.121027 60.25608) (xy 51.636874 59.447339) (xy 51.253105 58.416895)
-				(xy 50.222659 58.033127)
+				(xy 51.53524 58.841867) (xy 50.828133 58.13476) (xy 51.888793 59.195421) (xy 50.47289 59.19711)
+				(xy 50.474581 57.781207)
 			)
 		)
@@
 		(layer "B.Cu")
 		(hatch none 0.1)
-		(priority 30025)
+		(priority 30026)
 		(attr
 			(teardrop
@@
 		(layer "B.Cu")
 		(hatch none 0.1)
-		(priority 30092)
+		(priority 30131)
 		(attr
 			(teardrop
@@
 		(polygon
 			(pts
-				(xy 86.083485 47.969221) (xy 85.659221 48.393485) (xy 86.294463 49.687117) (xy 87.003431 49.313431)
-				(xy 87.377117 48.604463)
+				(xy 87.209408 49.095144) (xy 86.785144 49.519408) (xy 86.203852 49.388414) (xy 87.564978 49.874978)
+				(xy 86.203852 49.388414)
 			)
 		)
@@
 		(layer "B.Cu")
 		(hatch none 0.1)
-		(priority 30131)
+		(priority 30092)
 		(attr
 			(teardrop
@@
 		(polygon
 			(pts
-				(xy 87.209408 49.095144) (xy 86.785144 49.519408) (xy 86.203852 49.388414) (xy 87.564978 49.874978)
-				(xy 86.203852 49.388414)
+				(xy 86.083485 47.969221) (xy 85.659221 48.393485) (xy 86.294463 49.687117) (xy 87.003431 49.313431)
+				(xy 87.377117 48.604463)
 			)
 		)
@@
 		(layer "B.Cu")
 		(hatch none 0.1)
-		(priority 30112)
+		(priority 30132)
 		(attr
 			(teardrop
@@
 		(polygon
 			(pts
-				(xy 122.3 81.523467) (xy 121.7 81.523467) (xy 121.311003 82.750995) (xy 122 82.964467) (xy 122.688997 82.750995)
+				(xy 121.7 82.963467) (xy 122.3 82.963467) (xy 121.283467 83.030572) (xy 122 82.241) (xy 121.283467 83.030572)
 			)
 		)
@@
 		(layer "B.Cu")
 		(hatch none 0.1)
-		(priority 30132)
+		(priority 30111)
 		(attr
 			(teardrop
@@
 		(polygon
 			(pts
-				(xy 121.7 82.963467) (xy 122.3 82.963467) (xy 121.283467 83.030572) (xy 122 82.241) (xy 121.283467 83.030572)
+				(xy 122.3 81.523467) (xy 121.7 81.523467) (xy 121.311003 82.750995) (xy 122 82.964467) (xy 122.688997 82.750995)
 			)
 		)
@@
 		(layer "B.Cu")
 		(hatch none 0.1)
-		(priority 30111)
+		(priority 30112)
 		(attr
 			(teardrop
@@
 	)
 	(zone
-		(net "+15V")
-		(layer "B.Cu")
-		(hatch none 0.1)
-		(priority 30026)
-		(attr
-			(teardrop
-				(type padvia)
-			)
-		)
-		(connect_pads yes
-			(clearance 0)
-		)
-		(min_thickness 0.0254)
-		(fill yes
-			(island_removal_mode 1)
-		)
-		(polygon
-			(pts
-				(xy 94.525094 46.7322) (xy 95.2322 46.025094) (xy 94.368408 44.742485) (xy 93.746569 45.246569)
-				(xy 93.242485 45.868408)
-			)
-		)
-	)
-	(zone
 		(net "Net-(IC3B--)")
 		(layer "B.Cu")
@@
 	)
 	(zone
-		(net "Net-(IC4A-+)")
+		(net "+15V")
 		(layer "B.Cu")
 		(hatch none 0.1)
-		(priority 30087)
+		(priority 30013)
 		(attr
 			(teardrop
@@
 		(polygon
 			(pts
-				(xy 94.05 76.403852) (xy 93.45 76.403852) (xy 92.984448 77.767772) (xy 93.75 78.004852) (xy 94.515552 77.767772)
+				(xy 97.623852 55.67) (xy 97.623852 56.67) (xy 99.141586 56.966148) (xy 99.621 56.17) (xy 99.141586 55.373852)
 			)
 		)
 	)
 	(zone
-		(net "Net-(D4-K)")
+		(net "Net-(IC4A-+)")
 		(layer "B.Cu")
 		(hatch none 0.1)
-		(priority 30006)
+		(priority 30087)
 		(attr
 			(teardrop
@@
 		(polygon
 			(pts
-				(xy 68.846609 70.97) (xy 68.846609 70.37) (xy 67.202878 69.67) (xy 66.745609 70.67) (xy 67.202878 71.67)
+				(xy 94.05 76.403852) (xy 93.45 76.403852) (xy 92.984448 77.767772) (xy 93.75 78.004852) (xy 94.515552 77.767772)
 			)
 		)
 	)
 	(zone
-		(net "/PLANT/Vs")
+		(net "Net-(D4-K)")
 		(layer "B.Cu")
 		(hatch none 0.1)
-		(priority 30099)
+		(priority 30006)
 		(attr
 			(teardrop
@@
 		(polygon
 			(pts
-				(xy 72.689221 71.136515) (xy 73.113485 71.560779) (xy 74.377117 70.895537) (xy 74.033431 70.216569)
-				(xy 73.294463 69.812883)
+				(xy 68.846609 70.97) (xy 68.846609 70.37) (xy 67.202878 69.67) (xy 66.745609 70.67) (xy 67.202878 71.67)
 			)
 		)
 	)
 	(zone
-		(net "+15V")
+		(net "/PLANT/Vs")
 		(layer "B.Cu")
 		(hatch none 0.1)
-		(priority 30003)
+		(priority 30099)
 		(attr
 			(teardrop
@@
 		(polygon
 			(pts
-				(xy 85.096609 68.17) (xy 85.096609 67.17) (xy 83.452878 66.67) (xy 82.995609 67.67) (xy 83.452878 68.67)
+				(xy 72.689221 71.136515) (xy 73.113485 71.560779) (xy 74.377117 70.895537) (xy 74.033431 70.216569)
+				(xy 73.294463 69.812883)
 			)
 		)
@@
 		(layer "B.Cu")
 		(hatch none 0.1)
-		(priority 30013)
+		(priority 30003)
 		(attr
 			(teardrop
@@
 		(polygon
 			(pts
-				(xy 93.996148 56.67) (xy 93.996148 55.67) (xy 92.478414 55.373852) (xy 91.999 56.17) (xy 92.478414 56.966148)
+				(xy 85.096609 68.17) (xy 85.096609 67.17) (xy 83.452878 66.67) (xy 82.995609 67.67) (xy 83.452878 68.67)
 			)
 		)

Commit message: Editing some bug fixes in controller and plant.
Parts:
- C18: value 1uF -> 100uF; footprint Capacitor_THT:CP_Radial_Tantal_D5.0mm_P5.00mm -> Capacitor_THT:CP_Radial_Tantal_D8.0mm_P5.00mm
- C8: value 390pF -> 1nF
- R11: value 10kR -> 27kR
- R3: value 10kR -> 4.7kR

Commit message: Validating and verifying bug fix in controller, ready for v1.0.1  release.
Parts:
- R3: value 4.7kR -> 10kR
- R8: value 2.2kR -> 10kR

Commit message: Changing 1nF capacitor and buck-plant inductor footprints. Ready to release v1.0.1 (bug-fixes).
Parts:
- C8: footprint Capacitor_THT:C_Disc_D3.0mm_W2.0mm_P2.50mm -> Capacitor_THT:C_Rect_L7.2mm_W3.5mm_P5.00mm_FKS2_FKP2_MKS2_MKP2
- L1: footprint Inductor_THT:L_Toroid_Vertical_L16.0mm_W8.0mm_P7.62mm -> Inductor_THT:L_Toroid_Vertical_L25.4mm_W14.7mm_P12.20mm_Vishay_TJ5
- moved R22 11.8 mm to (93.8, 66.7)
- moved C7 6.80 mm to (103.8, 92.4), turned to 90 degrees
- moved R16 6.00 mm to (87.8, 75.3)
- moved C18 5.98 mm to (103.8, 97.0)
- moved L1 1.04 mm to (81.2, 93.5)
- turned R19 to 180 degrees
Routing:
- net +15V: track 231.7 -> 225.5 mm
- net Net-(C8-Pad2): track 34.0 -> 39.9 mm
- net Net-(IC4A--): track 8.77 -> 14.0 mm
- net /COMPENSATOR/Verr: track 35.5 -> 38.2 mm
- net Net-(IC4A-+): track 14.3 -> 16.3 mm
- net GND: vias 69 -> 79
- net (no net): vias 0 -> 4
Other:
- outline, holes or cut-outs redrawn
